File: DCDC-BASE-X2.brd (EAGLE design)
At the start: 50 x 70 mm, 7 parts

Commit message: Small fixes. Generated PNG preview. Generated CAM files.
Parts:
- LOGO2: value MFDECLOGO_L_20MM -> MFDECLOGO_L_10MM; device _my_logos:MFDEC_L_20MM -> _my_logos:MFDEC_L_10MM
- moved LOGO2 11.4 mm to (17.0, 29.0)
Routing:
- added copper zone on layer 1, net GND6
- added copper zone on layer 16, net GND6
- added copper zone on layer 1, net GND7
- added copper zone on layer 16, net GND7
- added copper zone on layer 1, net GND8
- added copper zone on layer 16, net GND8
- added copper zone on layer 1, net GND9
- added copper zone on layer 16, net GND9
Changed lines of the file:
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@@
 <attribute name="VALUE" x="38" y="9" size="0.6096" layer="27" font="vector"/>
 </element>
-<element name="LOGO2" library="_my_logos" package="MFDEC_L_20MM" value="MFDECLOGO_L_20MM" x="8" y="22" smashed="yes"/>
+<element name="LOGO2" library="_my_logos" package="MFDEC_L_10MM" value="MFDECLOGO_L_10MM" x="17" y="29" smashed="yes"/>
 </elements>
 <signals>
@@
 <via x="49" y="56" extent="1-16" drill="0.35"/>
 <via x="49" y="19" extent="1-16" drill="0.35"/>
+<via x="47" y="37" extent="1-16" drill="0.35"/>
+<via x="47" y="33" extent="1-16" drill="0.35"/>
 </signal>
 <signal name="VOUT1" airwireshidden="yes">
@@
 </polygon>
 </signal>
+<signal name="GND6" airwireshidden="yes">
+<polygon width="0.1524" layer="1" pour="cutout">
+<vertex x="42" y="44" curve="-180"/>
+<vertex x="42" y="48" curve="-180"/>
+</polygon>
+<polygon width="0.1524" layer="16" pour="cutout">
+<vertex x="42" y="44" curve="-180"/>
+<vertex x="42" y="48" curve="-180"/>
+</polygon>
+</signal>
+<signal name="GND7" airwireshidden="yes">
+<polygon width="0.1524" layer="1" pour="cutout">
+<vertex x="42" y="22" curve="-180"/>
+<vertex x="42" y="26" curve="-180"/>
+</polygon>
+<polygon width="0.1524" layer="16" pour="cutout">
+<vertex x="42" y="22" curve="-180"/>
+<vertex x="42" y="26" curve="-180"/>
+</polygon>
+</signal>
+<signal name="GND8" airwireshidden="yes">
+<polygon width="0.1524" layer="1" pour="cutout">
+<vertex x="8" y="22" curve="-180"/>
+<vertex x="8" y="26" curve="-180"/>
+</polygon>
+<polygon width="0.1524" layer="16" pour="cutout">
+<vertex x="8" y="22" curve="-180"/>
+<vertex x="8" y="26" curve="-180"/>
+</polygon>
+</signal>
+<signal name="GND9" airwireshidden="yes">
+<polygon width="0.1524" layer="1" pour="cutout">
+<vertex x="42" y="4" curve="-180"/>
+<vertex x="42" y="8" curve="-180"/>
+</polygon>
+<polygon width="0.1524" layer="16" pour="cutout">
+<vertex x="42" y="4" curve="-180"/>
+<vertex x="42" y="8" curve="-180"/>
+</polygon>
+</signal>
