File: DCDC-BASE-X2.sch (EAGLE design)
At the start: 7 parts

Commit message: Small fixes. Generated PNG preview. Generated CAM files.
Parts:
- LOGO2: value MFDECLOGO_L_20MM -> MFDECLOGO_L_10MM; device _my_logos:MFDECLOGO_L_20MM -> _my_logos:MFDECLOGO_L_10MM
Changed lines of the file:
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@@
 <part name="GND4" library="SparkFun-PowerSymbols" library_urn="urn:adsk.eagle:library:530" deviceset="GND" device=""/>
 <part name="GND5" library="SparkFun-PowerSymbols" library_urn="urn:adsk.eagle:library:530" deviceset="GND" device=""/>
-<part name="LOGO2" library="_my_logos" deviceset="MFDECLOGO" device="_L_20MM" value="MFDECLOGO_L_20MM"/>
+<part name="LOGO2" library="_my_logos" deviceset="MFDECLOGO" device="_L_10MM" value="MFDECLOGO_L_10MM"/>
 </parts>
 <sheets>
