File: DCDC-BASE-X2B.brd (EAGLE design)
At the start: 50 x 70 mm, 7 parts

Commit message: Moved some stuff around on x2 boards. Generated CAM files. Generated PNG preview.
Parts:
- moved CN1 2.00 mm to (30.0, 4.00)
- moved CN2 2.00 mm to (19.0, 3.00)
Changed lines of the file:
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@@
 <hole x="47" y="3" drill="3.1"/>
 <text x="40" y="36" size="1.6764" layer="22" font="vector" ratio="20" rot="MR0">DCDC-BASE-X2B-0010</text>
-<text x="27.6" y="2" size="0.8128" layer="21" font="vector" rot="R90">GND</text>
+<text x="25.6" y="2" size="0.8128" layer="21" font="vector" rot="R90">GND</text>
 <text x="26" y="65.1" size="0.8128" layer="21" font="vector" rot="R180">GND</text>
 <text x="47" y="28" size="1.27" layer="22" font="vector" rot="MR90">(c) Andriy Golovnya</text>
 <text x="40" y="33" size="1.27" layer="22" font="vector" rot="MR0">Base x2 Board for Converters</text>
-<text x="24.6" y="0.6" size="0.8128" layer="22" font="vector" rot="MR0">GND</text>
+<text x="22.6" y="0.6" size="0.8128" layer="22" font="vector" rot="MR0">GND</text>
 <text x="26" y="68.5" size="0.8128" layer="22" font="vector" rot="MR0">GND</text>
 <text x="44" y="28" size="1.27" layer="22" font="vector" rot="MR90">http://redscorp.net</text>
-<text x="28.5" y="5.3" size="1.27" layer="22" font="vector" rot="MR0">INPUT</text>
+<text x="26.5" y="5.3" size="1.27" layer="22" font="vector" rot="MR0">INPUT</text>
 <text x="28.1" y="63.4" size="1.27" layer="22" font="vector" rot="MR0">OUTPUT</text>
 <wire x1="0" y1="68" x2="0" y2="2" width="0" layer="20"/>
@@
 <text x="21.5" y="68.5" size="0.8128" layer="22" font="vector" rot="MR0">VOUT1</text>
 <text x="31.8" y="68.5" size="0.8128" layer="22" font="vector" rot="MR0">VOUT2</text>
-<text x="19.4" y="0.6" size="0.8128" layer="22" font="vector" rot="MR0">VIN</text>
-<text x="15.2" y="2.1" size="0.8128" layer="21" font="vector" rot="R90">VIN</text>
+<text x="17.4" y="0.6" size="0.8128" layer="22" font="vector" rot="MR0">VIN</text>
+<text x="13.2" y="2.1" size="0.8128" layer="21" font="vector" rot="R90">VIN</text>
 <text x="16.6" y="65.8" size="0.8128" layer="21" font="vector" rot="R90">VOUT1</text>
 <text x="34.2" y="65.9" size="0.8128" layer="21" font="vector" rot="R90">VOUT2</text>
 <hole x="3" y="3" drill="3.1"/>
-<text x="7" y="5" size="1.778" layer="21" font="vector">INPUT</text>
+<text x="6" y="5" size="1.778" layer="21" font="vector">INPUT</text>
 <text x="6" y="63" size="1.778" layer="21" font="vector">OUTPUT</text>
 <text x="48" y="45" size="1.778" layer="21" font="vector" rot="R90">Module 1</text>
-<text x="48" y="14" size="1.778" layer="21" font="vector" rot="R90">Module 2</text>
+<text x="48" y="15" size="1.778" layer="21" font="vector" rot="R90">Module 2</text>
 </plain>
 <attributes>
@@
 </autorouter>
 <elements>
-<element name="CN1" library="con-jack" library_urn="urn:adsk.eagle:library:154" package="SPC4078" package3d_urn="urn:adsk.eagle:package:7494/1" value="" x="32" y="4" smashed="yes" rot="R90">
-<attribute name="MF" value="" x="38.35" y="34.48" size="1.778" layer="27" rot="R90" display="off"/>
-<attribute name="MPN" value="" x="38.35" y="34.48" size="1.778" layer="27" rot="R90" display="off"/>
-<attribute name="NAME" x="26.92" y="-6.16" size="0.6096" layer="25" font="vector" rot="R90"/>
-<attribute name="OC_FARNELL" value="unknown" x="38.35" y="34.48" size="1.778" layer="27" rot="R90" display="off"/>
-<attribute name="OC_NEWARK" value="unknown" x="38.35" y="34.48" size="1.778" layer="27" rot="R90" display="off"/>
-<attribute name="POPULARITY" value="3" x="38.35" y="34.48" size="1.778" layer="27" rot="R90" display="off"/>
-<attribute name="VALUE" x="38.35" y="-6.16" size="1.27" layer="27" rot="R90"/>
+<element name="CN1" library="con-jack" library_urn="urn:adsk.eagle:library:154" package="SPC4078" package3d_urn="urn:adsk.eagle:package:7494/1" value="" x="30" y="4" smashed="yes" rot="R90">
+<attribute name="MF" value="" x="36.35" y="34.48" size="1.778" layer="27" rot="R90" display="off"/>
+<attribute name="MPN" value="" x="36.35" y="34.48" size="1.778" layer="27" rot="R90" display="off"/>
+<attribute name="NAME" x="24.92" y="-6.16" size="0.6096" layer="25" font="vector" rot="R90"/>
+<attribute name="OC_FARNELL" value="unknown" x="36.35" y="34.48" size="1.778" layer="27" rot="R90" display="off"/>
+<attribute name="OC_NEWARK" value="unknown" x="36.35" y="34.48" size="1.778" layer="27" rot="R90" display="off"/>
+<attribute name="POPULARITY" value="3" x="36.35" y="34.48" size="1.778" layer="27" rot="R90" display="off"/>
+<attribute name="VALUE" x="36.35" y="-6.16" size="1.27" layer="27" rot="R90"/>
 </element>
-<element name="CN2" library="Wurth_Connectors_WR-TBL Rising Cage Clamp" library_urn="urn:adsk.eagle:library:16280519" package="691213510002" package3d_urn="urn:adsk.eagle:package:16248575/2" value="" x="21" y="3" smashed="yes">
-<attribute name="IR-UL" value="14A" x="21" y="3" size="1.778" layer="27" display="off"/>
-<attribute name="IR-VDE" value="14A" x="21" y="3" size="1.778" layer="27" display="off"/>
-<attribute name="NAME" x="22.27" y="-2.4" size="0.6096" layer="25" font="vector" align="bottom-center"/>
-<attribute name="PART-NUMBER" value=" 691213510002 " x="21" y="3" size="1.778" layer="27" display="off"/>
-<attribute name="PINS" value=" 2 " x="21" y="3" size="1.778" layer="27" display="off"/>
-<attribute name="PITCH" value="5.08mm" x="21" y="3" size="1.778" layer="27" display="off"/>
-<attribute name="TYPE" value="Horizontal" x="21" y="3" size="1.778" layer="27" display="off"/>
-<attribute name="VALUE" x="22.27" y="6.9" size="0.6096" layer="27" font="vector" align="bottom-center"/>
-<attribute name="WIRE" value="14 to 30 (AWG) 2.08 to 0.0509 (mm²)" x="21" y="3" size="1.778" layer="27" display="off"/>
-<attribute name="WORKING-VOLTAGE-UL" value="300V (AC)" x="21" y="3" size="1.778" layer="27" display="off"/>
-<attribute name="WORKING-VOLTAGE-VDE" value="250V (AC)" x="21" y="3" size="1.778" layer="27" display="off"/>
+<element name="CN2" library="Wurth_Connectors_WR-TBL Rising Cage Clamp" library_urn="urn:adsk.eagle:library:16280519" package="691213510002" package3d_urn="urn:adsk.eagle:package:16248575/2" value="" x="19" y="3" smashed="yes">
+<attribute name="IR-UL" value="14A" x="19" y="3" size="1.778" layer="27" display="off"/>
+<attribute name="IR-VDE" value="14A" x="19" y="3" size="1.778" layer="27" display="off"/>
+<attribute name="NAME" x="18.97" y="-2.3" size="0.6096" layer="25" font="vector" align="bottom-center"/>
+<attribute name="PART-NUMBER" value=" 691213510002 " x="19" y="3" size="1.778" layer="27" display="off"/>
+<attribute name="PINS" value=" 2 " x="19" y="3" size="1.778" layer="27" display="off"/>
+<attribute name="PITCH" value="5.08mm" x="19" y="3" size="1.778" layer="27" display="off"/>
+<attribute name="TYPE" value="Horizontal" x="19" y="3" size="1.778" layer="27" display="off"/>
+<attribute name="VALUE" x="20.27" y="6.9" size="0.6096" layer="27" font="vector" align="bottom-center"/>
+<attribute name="WIRE" value="14 to 30 (AWG) 2.08 to 0.0509 (mm²)" x="19" y="3" size="1.778" layer="27" display="off"/>
+<attribute name="WORKING-VOLTAGE-UL" value="300V (AC)" x="19" y="3" size="1.778" layer="27" display="off"/>
+<attribute name="WORKING-VOLTAGE-VDE" value="250V (AC)" x="19" y="3" size="1.778" layer="27" display="off"/>
 </element>
 <element name="CN3" library="Wurth_Connectors_WR-TBL Rising Cage Clamp" library_urn="urn:adsk.eagle:library:16280519" package="691213510003" package3d_urn="urn:adsk.eagle:package:16248576/2" value="" x="25" y="67" smashed="yes" rot="R180">
 <attribute name="IR-UL" value="14A" x="25" y="67" size="1.778" layer="27" rot="R180" display="off"/>
 <attribute name="IR-VDE" value="14A" x="25" y="67" size="1.778" layer="27" rot="R180" display="off"/>
-<attribute name="NAME" x="23.73" y="72.4" size="0.6096" layer="25" font="vector" rot="R180" align="bottom-center"/>
+<attribute name="NAME" x="25.03" y="72.3" size="0.6096" layer="25" font="vector" rot="R180" align="bottom-center"/>
 <attribute name="PART-NUMBER" value=" 691213510003 " x="25" y="67" size="1.778" layer="27" rot="R180" display="off"/>
 <attribute name="PINS" value=" 3 " x="25" y="67" size="1.778" layer="27" rot="R180" display="off"/>
@@
 <contactref element="MOD2" pad="VIN"/>
 <polygon width="0.3048" layer="1" thermals="no">
-<vertex x="35" y="8"/>
-<vertex x="35" y="6"/>
-<vertex x="33" y="4"/>
-<vertex x="22" y="4"/>
-<vertex x="20" y="2"/>
+<vertex x="33" y="8"/>
+<vertex x="33" y="6"/>
+<vertex x="31" y="4"/>
+<vertex x="20" y="4"/>
+<vertex x="18" y="2"/>
 <vertex x="9" y="2"/>
 <vertex x="1" y="10"/>
@@
 <via x="15" y="37" extent="1-16" drill="0.35"/>
 <via x="17" y="69" extent="1-16" drill="0.35"/>
-<via x="17" y="1" extent="1-16" drill="0.35"/>
-<via x="33" y="1" extent="1-16" drill="0.35"/>
+<via x="15" y="1" extent="1-16" drill="0.35"/>
+<via x="31" y="1" extent="1-16" drill="0.35"/>
 <via x="12" y="9" extent="1-16" drill="0.35"/>
 <via x="1" y="51" extent="1-16" drill="0.35"/>
@@
 <via x="6" y="61" extent="1-16" drill="0.35"/>
 <via x="43" y="38" extent="1-16" drill="0.35"/>
-<via x="22" y="2" extent="1-16" drill="0.35"/>
-<via x="25" y="3" extent="1-16" drill="0.35"/>
-<via x="24" y="1" extent="1-16" drill="0.35"/>
-<via x="34" y="3" extent="1-16" drill="0.35"/>
-<via x="37" y="7" extent="1-16" drill="0.35"/>
-<via x="37" y="1" extent="1-16" drill="0.35"/>
-<via x="29" y="3" extent="1-16" drill="0.35"/>
+<via x="20" y="2" extent="1-16" drill="0.35"/>
+<via x="23" y="3" extent="1-16" drill="0.35"/>
+<via x="22" y="1" extent="1-16" drill="0.35"/>
+<via x="32" y="3" extent="1-16" drill="0.35"/>
+<via x="35" y="7" extent="1-16" drill="0.35"/>
+<via x="35" y="1" extent="1-16" drill="0.35"/>
+<via x="28" y="3" extent="1-16" drill="0.35"/>
 <via x="19" y="63" extent="1-16" drill="0.35"/>
 <via x="12" y="54" extent="1-16" drill="0.35"/>
@@
 <via x="45" y="8" extent="1-16" drill="0.35"/>
 <via x="12" y="23" extent="1-16" drill="0.35"/>
+<via x="37" y="6" extent="1-16" drill="0.35"/>
+<via x="37" y="2" extent="1-16" drill="0.35"/>
+<via x="38" y="4" extent="1-16" drill="0.35"/>
+<via x="26" y="1" extent="1-16" drill="0.35"/>
 </signal>
 <signal name="VOUT1" airwireshidden="yes">
