File: DCDC-17VXV5A.brd (EAGLE design)
At the start: 40 x 24 mm, 36 parts, among them Q10 NMOSFET, Q9 NMOSFET, U1 LM3150MHX/NOPB

Commit message: Changed LEDs resistor. Generated CAM filers. Generated PNG preview. Generated PDF schematics. Updated description.
Parts:
- R1: value 2k -> 10k
Changed lines of the file:
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@@
 <drawing>
 <settings>
-<setting alwaysvectorfont="yes"/>
+<setting alwaysvectorfont="no"/>
 <setting verticaltext="up"/>
 </settings>
@@
 <attribute name="VALUE" x="31" y="20" size="0.6096" layer="27" font="vector" rot="R270"/>
 </element>
-<element name="R1" library="rcl" library_urn="urn:adsk.eagle:library:334" package="R0603" package3d_urn="urn:adsk.eagle:package:23555/3" value="2k" x="33" y="22" smashed="yes" rot="R270">
+<element name="R1" library="rcl" library_urn="urn:adsk.eagle:library:334" package="R0603" package3d_urn="urn:adsk.eagle:package:23555/3" value="10k" x="33" y="22" smashed="yes" rot="R270">
 <attribute name="NAME" x="33.635" y="22.635" size="0.6096" layer="25" font="vector" rot="R270"/>
 <attribute name="POPULARITY" value="70" x="33" y="22" size="1.778" layer="27" font="vector" rot="R270" display="off"/>
