File: DCDC-12V5V1A.brd (EAGLE design)
At the start: 40 x 24 mm, 34 parts, among them U1 TPS63060DSCT

Commit message: Changed L1 inductor from 1uH to 1.5uH for higher output current stability. Generated PDF schematics. Updated BoM file.
Parts:
- L1: value 1uH -> 1.5uH
Changed lines of the file:
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@@
 <attribute name="VALUE" x="16.35" y="6.8" size="0.6096" layer="27" rot="R270"/>
 </element>
-<element name="L1" library="Wurth_Power Magnetics_WE-LQS" library_urn="urn:adsk.eagle:library:14283646" package="WE-LQS_4018" package3d_urn="urn:adsk.eagle:package:13009659/3" value="1uH" x="16" y="15" smashed="yes" rot="R180">
+<element name="L1" library="Wurth_Power Magnetics_WE-LQS" library_urn="urn:adsk.eagle:library:14283646" package="WE-LQS_4018" package3d_urn="urn:adsk.eagle:package:13009659/3" value="1.5uH" x="16" y="15" smashed="yes" rot="R180">
 <attribute name="DATASHEET-URL" value="https://www.we-online.com/redexpert/spec/74404042010?ae" x="16" y="15" size="1.778" layer="27" rot="R180" display="off"/>
 <attribute name="FRES" value="120MHz" x="16" y="15" size="1.778" layer="27" rot="R180" display="off"/>
